Commit message: launch files cleaned - TODO: create launch files for pick and place nodes

File: src/franka_ros/franka_description/robots/common/utils.xacro (robot description, xacro)
@@ -224,5 +224,6 @@
                          soft_upper_limit="${limits.upper}" />
   </xacro:macro>
-  <!-- Colourize the links -->
+  <!-- Colourize the and add friction to the links, the fingers have seperate friction values
+  set with the gazebo-friction macro in the franka_robot.xacro file -->
   <xacro:macro name="panda_gazebo" params="arm_id">
   <xacro:macro name="arm_gazebo" params="link">
@@ -234,4 +235,11 @@
       </xacro:macro>
       <xacro:macro name="hand_gazebo" params="link">
+          <gazebo reference="${link}">
+              <material>Gazebo/Grey</material>
+              <mu1>0.2</mu1>
+              <mu2>0.2</mu2>
+          </gazebo>
+      </xacro:macro>
+      <xacro:macro name="hand_gazebo_no_friction" params="link">
           <gazebo reference="${link}">
               <material>Gazebo/Grey</material>
@@ -248,6 +256,6 @@
       <xacro:hand_gazebo link="${arm_id}_link8"/>
       <xacro:hand_gazebo link="${arm_id}_hand"/>
-      <xacro:hand_gazebo link="${arm_id}_rightfinger"/>
-      <xacro:hand_gazebo link="${arm_id}_leftfinger"/>
+      <xacro:hand_gazebo_no_friction link="${arm_id}_rightfinger"/>
+      <xacro:hand_gazebo_no_friction link="${arm_id}_leftfinger"/>
   </xacro:macro>
 </robot>

File: src/franka_ros/franka_description/robots/panda/panda.urdf.xacro (robot description, xacro)
@@ -19,4 +19,6 @@
   <!-- If `gazebo` arg is set and `parent` not empty, what rotation offset between `parent` & $(arm_id)_link0 -->
   <xacro:arg name="rpy" default="0 0 0" />
+  <!-- additional args -->
+  <xacro:arg name="use_cameras" default="false" />
   <xacro:franka_robot arm_id="$(arg arm_id)"
                       joint_limits="${xacro.load_yaml('$(find franka_description)/robots/panda/joint_limits.yaml')}"
@@ -29,17 +31,13 @@
                       rpy="$(arg rpy)">
   </xacro:franka_robot>
+  <!-- colourize and add friction to panda arm -->
   <xacro:panda_gazebo arm_id="$(arg arm_id)" />
-<!-- Scene view (D435 optimal range 0.3m-10m) -->
-<xacro:if value="$(optenv INCLUDE_D435_CAMERA false)">
-  <xacro:include filename="$(find realsense_gazebo_description)/urdf/_d435.urdf.xacro"/>
-  <xacro:sensor_d435  parent="panda_link0" name="D435_camera1" topics_ns="D435_camera1" align_depth="true" visualize="true" enable_pointCloud="true" clip_distance="10">
-    <origin xyz="0.0 0.4 0.425" rpy="0.0 0.26 -0.58875"/>
-  </xacro:sensor_d435>
-</xacro:if>
- <!-- Scene view (D435 optimal range 0.3m-10m) [Comment out when running roslaunch panda_moveit run_sim.launch]-->
- <!-- <xacro:include filename="$(find realsense_gazebo_description)/urdf/_d435.urdf.xacro"/>
-  <xacro:sensor_d435  parent="panda_link0" name="D435_camera1" topics_ns="D435_camera1" align_depth="true" visualize="true" enable_pointCloud="true" clip_distance="10">
-    <origin xyz="0.0 0.4 0.425" rpy="0.0 0.26 -0.58875"/>
- </xacro:sensor_d435> -->
+  <!-- Scene view (D435 optimal range 0.3m-10m) -->
+  <xacro:if value="$(arg use_cameras)">
+    <xacro:include filename="$(find realsense_gazebo_description)/urdf/_d435.urdf.xacro"/>
+    <xacro:sensor_d435  parent="panda_link0" name="D435_camera1" topics_ns="D435_camera1" align_depth="true" visualize="true" enable_pointCloud="true" clip_distance="10">
+      <origin xyz="0.0 0.4 0.425" rpy="0.0 0.26 -0.58875"/>
+    </xacro:sensor_d435>
+  </xacro:if>
   <!-- Camera on hand view -->
   <!-- <xacro:include filename="$(find realsense_gazebo_description)/urdf/_d435.urdf.xacro"/>
