Commit message: small changes- TODO: create launch arguments for camera

File: src/franka_ros/franka_description/robots/panda/panda.urdf.xacro (robot description, xacro)
@@ -19,5 +19,4 @@
   <!-- If `gazebo` arg is set and `parent` not empty, what rotation offset between `parent` & $(arm_id)_link0 -->
   <xacro:arg name="rpy" default="0 0 0" />
-  <!-- <xacro:panda_gazebo arm_id="panda"/> -->
   <xacro:franka_robot arm_id="$(arg arm_id)"
                       joint_limits="${xacro.load_yaml('$(find franka_description)/robots/panda/joint_limits.yaml')}"
@@ -30,4 +29,14 @@
                       rpy="$(arg rpy)">
   </xacro:franka_robot>
+ <!-- Scene view (D435 optimal range 0.3m-10m) [Comment out when running roslaunch panda_moveit run_sim.launch]-->
+ <!-- <xacro:include filename="$(find realsense_gazebo_description)/urdf/_d435.urdf.xacro"/>
+  <xacro:sensor_d435  parent="panda_link0" name="D435_camera1" topics_ns="D435_camera1" align_depth="true" visualize="true" enable_pointCloud="true" clip_distance="10">
+    <origin xyz="0.0 0.4 0.425" rpy="0.0 0.26 -0.58875"/>
+ </xacro:sensor_d435> -->
+ <!-- Scene view (D435 optimal range 0.3m-10m) [Comment out when running roslaunch panda_moveit run_sim.launch]-->
+ <!-- <xacro:include filename="$(find realsense_gazebo_description)/urdf/_d435.urdf.xacro"/>
+  <xacro:sensor_d435  parent="panda_link0" name="D435_camera1" topics_ns="D435_camera1" align_depth="true" visualize="true" enable_pointCloud="true" clip_distance="10">
+    <origin xyz="0.0 0.4 0.425" rpy="0.0 0.26 -0.58875"/>
+ </xacro:sensor_d435> -->
   <!-- Camera on hand view -->
   <!-- <xacro:include filename="$(find realsense_gazebo_description)/urdf/_d435.urdf.xacro"/>
@@ -44,9 +53,4 @@
   <origin xyz="0.045 0.0 0.055" rpy="0.0 -1.34 0.0"/>
   </xacro:sensor_d435> -->
- <!-- Scene view (D435 optimal range 0.3m-10m) [Comment out when running roslaunch panda_moveit run_sim.launch]-->
- <!-- <xacro:include filename="$(find realsense_gazebo_description)/urdf/_d435.urdf.xacro"/>
-  <xacro:sensor_d435  parent="panda_link0" name="D435_camera1" topics_ns="D435_camera1" align_depth="true" visualize="true" enable_pointCloud="true" clip_distance="10">
-    <origin xyz="0.0 0.4 0.425" rpy="0.0 0.26 -0.58875"/>
- </xacro:sensor_d435> -->
   <!-- Scene view (D435 optimal range 0.3m-10m) -->
   <!-- <xacro:include filename="$(find realsense_gazebo_description)/urdf/_d435.urdf.xacro"/>

Commit message: update camera plugin and launch files

File: src/franka_ros/franka_description/robots/panda/panda.urdf.xacro (robot description, xacro)
@@ -20,5 +20,6 @@
   <xacro:arg name="rpy" default="0 0 0" />
   <!-- additional args -->
-  <xacro:arg name="use_cameras" default="false" />
+  <xacro:arg name="use_camera1" default="false" />
+  <xacro:arg name="use_camera2" default="false" />
   <xacro:franka_robot arm_id="$(arg arm_id)"
                       joint_limits="${xacro.load_yaml('$(find franka_description)/robots/panda/joint_limits.yaml')}"
@@ -34,24 +35,38 @@
   <xacro:panda_gazebo arm_id="$(arg arm_id)" />
   <!-- Scene view (D435 optimal range 0.3m-10m) -->
-  <xacro:if value="$(arg use_cameras)">
+  <xacro:if value="$(arg use_camera1)">
     <xacro:include filename="$(find realsense_gazebo_description)/urdf/_d435.urdf.xacro"/>
-    <xacro:sensor_d435  parent="panda_link0" name="D435_camera1" topics_ns="D435_camera1" align_depth="true" visualize="true" enable_pointCloud="true" clip_distance="10">
+    <xacro:sensor_d435  parent="panda_link0"
+                        name="D435_camera1"
+                        topics_ns="D435_camera1"
+                        align_depth="true"
+                        visualize="true"
+                        enable_pointCloud="true"
+                        clip_distance="10">
       <origin xyz="0.0 0.4 0.425" rpy="0.0 0.26 -0.58875"/>
     </xacro:sensor_d435>
   </xacro:if>
   <!-- Camera on hand view -->
-  <!-- <xacro:include filename="$(find realsense_gazebo_description)/urdf/_d435.urdf.xacro"/>
-  <xacro:sensor_d435 parent="panda_hand"
-                     name="D435_camera"
-                     topics_ns="camera"
-                     align_depth="true"
-                     visualize="true"
-                     enable_pointCloud="true"
-                     depth_width="640"
-                     depth_height="480"
-                     color_width="640"
-                     color_height="480">
-  <origin xyz="0.045 0.0 0.055" rpy="0.0 -1.34 0.0"/>
-  </xacro:sensor_d435> -->
+  <xacro:if value="$(arg use_camera2)">
+    <xacro:include filename="$(find realsense_gazebo_description)/urdf/_d435.urdf.xacro"/>
+    <xacro:sensor_d435  parent="panda_link0"
+                        name="D435_camera1"
+                        topics_ns="D435_camera1"
+                        align_depth="true"
+                        visualize="true"
+                        enable_pointCloud="true"
+                        clip_distance="10">
+      <origin xyz="0.0 0.4 0.425" rpy="0.0 0.26 -0.58875"/>
+    </xacro:sensor_d435>
+    <xacro:include filename="$(find realsense_gazebo_description)/urdf/_d435.urdf.xacro"/>
+    <xacro:sensor_d435  parent="panda_hand"
+                        name="D435_camera2"
+                        topics_ns="D435_camera2"
+                        align_depth="true"
+                        visualize="true" >
+      <origin xyz="0.045 0.0 -0.05" rpy="3.1415 -1.34 0.0"/>
+      <!-- <origin xyz="0.045 0.0 0.055" rpy="3.1415 -1.34 0.0"/> -->
+    </xacro:sensor_d435>
+   </xacro:if>
   <!-- Scene view (D435 optimal range 0.3m-10m) -->
   <!-- <xacro:include filename="$(find realsense_gazebo_description)/urdf/_d435.urdf.xacro"/>

File: src/realsense_gazebo_description/urdf/_d435i.gazebo.xacro (robot description, xacro)
@@ -227,5 +227,6 @@
       	<infrared2OpticalframeName>${infrared2_optical_frame}</infrared2OpticalframeName>
         <!-- Depth camera settings -->
-      	<rangeMinDepth>0.2</rangeMinDepth>
+      	<!-- <rangeMinDepth>0.2</rangeMinDepth> -->
+        <rangeMinDepth>0.1</rangeMinDepth>
         <xacro:unless value="${clip_distance > 0.0}">
       	  <rangeMaxDepth>10.0</rangeMaxDepth>
